Commit message: something wrong with chassis

File: twizy_sensor_kit_description/urdf/VLP-16.urdf.xacro (robot description, xacro)
@@ -18,10 +18,10 @@
             <visual>
                 <geometry>
-                    <mesh filename="file:///$(find vehicle_model)/meshes/VLP16_base_1.dae" />
+                    <mesh filename="file:///$(find twizy_sensor_kit_description)/meshes/VLP16_base_1.dae" />
                 </geometry>
             </visual>
             <visual>
                 <geometry>
-                    <mesh filename="file:///$(find vehicle_model)/meshes/VLP16_base_2.dae" />
+                    <mesh filename="file:///$(find twizy_sensor_kit_description)/meshes/VLP16_base_2.dae" />
                 </geometry>
             </visual>
@@ -47,5 +47,5 @@
                 <origin xyz="0 0 -0.0377" />
                 <geometry>
-                    <mesh filename="file:///$(find vehicle_model)/meshes/VLP16_scan.dae" />
+                    <mesh filename="file:///$(find twizy_sensor_kit_description)/meshes/VLP16_scan.dae" />
                 </geometry>
             </visual>

File: twizy_sensor_kit_description/urdf/cameras.urdf.xacro (robot description, xacro)
@@ -6,9 +6,9 @@
 -->
 <robot xmlns:xacro="http://www.ros.org/wiki/xacro" name="blackfly_camera">
-    <xacro:macro name="blackfly_camera" params="frlr_prefix lrc_prefix *origin">
+    <xacro:macro name="blackfly_camera" params="frlr_prefix lrc_prefix origin parent">
     <joint name="${frlr_prefix}_${lrc_prefix}_camera_joint" type="fixed">
       <axis xyz="0 1 0" />
-      <xacro:insert_block name="origin"/>
-      <parent link="chassis"/>
+      <origin xyz="${origin.split()[0]} ${origin.split()[1]} ${origin.split()[2]}" rpy="${origin.split()[3]} ${origin.split()[4]} ${origin.split()[5]}"/>
+      <parent link="${parent}"/>
       <child link="${frlr_prefix}_${lrc_prefix}_camera_link"/>
     </joint>

File: twizy_sensor_kit_description/urdf/sensor_kit.xacro (robot description, xacro)
@@ -4,9 +4,12 @@
     <xacro:include filename="$(find twizy_sensor_kit_description)/urdf/cameras.urdf.xacro"/>
     <xacro:include filename="$(find twizy_vehicle_description)/urdf/bases/sd_twizy_body.urdf.xacro"/>
-    <xacro:include filename="$(find vehicle_model)/urdf/wheels/sd_twizy_suspension.urdf.xacro" />
+    <xacro:include filename="$(find twizy_vehicle_description)/urdf/wheels/sd_twizy_suspension.urdf.xacro" />
     <xacro:arg name="config_dir" default="$(find twizy_sensor_kit_description)/config"/>
+    <!--
     <xacro:property name="calibration" value="${xacro.load_yaml('$(arg config_dir)/sensor_kit_calibration.yaml')}"/>
+-->
+    <xacro:property name="calibration" value="${xacro.load_yaml('/home/robin/Documents/autoware/install/twizy_sensor_kit_description/share/twizy_sensor_kit_description/config/sensor_kit_calibration.yaml')}"/>
     <!-- chassis from sd_twizy_base -->
-    <xacro:sd_twizy_base name="sd_twizy"/>
+    <xacro:sd_twizy_base name="twizy_vehicle"/>
       <!-- Camera -->
     <xacro:blackfly_camera frlr_prefix="front" lrc_prefix="left" parent="chassis"

File: twizy_sensor_kit_description/urdf/sensors.xacro (robot description, xacro)
@@ -2,5 +2,8 @@
 <robot name="vehicle" xmlns:xacro="http://ros.org/wiki/xacro">
   <xacro:arg name="config_dir" default="$(find twizy_sensor_kit_description)/config"/>
-  <xacro:property name="calibration" value="${xacro.load_yaml('$(arg config_dir)/sensors_calibration.yaml')}"/>
+    <!--
+    <xacro:property name="calibration" value="${xacro.load_yaml('$(arg config_dir)/sensor_kit_calibration.yaml')}"/>
+-->
+    <xacro:property name="calibration" value="${xacro.load_yaml('/home/robin/Documents/autoware/install/twizy_sensor_kit_description/share/twizy_sensor_kit_description/config/sensor_kit_calibration.yaml')}"/>
   <!-- Sensor Kit -->
   <!-- Assuming sensor_kit_macro has been updated to place sensors relative to chassis_joint -->

Commit message: fixed twizy model

File: twizy_sensor_kit_description/urdf/VLP-16.urdf.xacro (robot description, xacro)
@@ -18,10 +18,10 @@
             <visual>
                 <geometry>
-                    <mesh filename="file:///$(find twizy_sensor_kit_description)/meshes/VLP16_base_1.dae" />
+                    <mesh filename="file:///$(find twizy_vehicle_description)/mesh/VLP16_base_1.dae" />
                 </geometry>
             </visual>
             <visual>
                 <geometry>
-                    <mesh filename="file:///$(find twizy_sensor_kit_description)/meshes/VLP16_base_2.dae" />
+                    <mesh filename="file:///$(find twizy_vehicle_description)/mesh/VLP16_base_2.dae" />
                 </geometry>
             </visual>
@@ -47,5 +47,5 @@
                 <origin xyz="0 0 -0.0377" />
                 <geometry>
-                    <mesh filename="file:///$(find twizy_sensor_kit_description)/meshes/VLP16_scan.dae" />
+                    <mesh filename="file:///$(find twizy_vehicle_description)/mesh/VLP16_scan.dae" />
                 </geometry>
             </visual>

File: twizy_sensor_kit_description/urdf/cameras.urdf.xacro (robot description, xacro)
@@ -6,4 +6,7 @@
 -->
 <robot xmlns:xacro="http://www.ros.org/wiki/xacro" name="blackfly_camera">
+    <material name="red">
+     <color rgba="1 0 0 1"/> <!-- Red color; adjust RGBA values as needed -->
+    </material>
     <xacro:macro name="blackfly_camera" params="frlr_prefix lrc_prefix origin parent">
     <joint name="${frlr_prefix}_${lrc_prefix}_camera_joint" type="fixed">

File: twizy_sensor_kit_description/urdf/sensor_kit.xacro (robot description, xacro)
@@ -4,5 +4,5 @@
     <xacro:include filename="$(find twizy_sensor_kit_description)/urdf/cameras.urdf.xacro"/>
     <xacro:include filename="$(find twizy_vehicle_description)/urdf/bases/sd_twizy_body.urdf.xacro"/>
-    <xacro:include filename="$(find twizy_vehicle_description)/urdf/wheels/sd_twizy_suspension.urdf.xacro" />
+    <!--<xacro:include filename="$(find twizy_vehicle_description)/urdf/wheels/sd_twizy_suspension.urdf.xacro" /> -->
     <xacro:arg name="config_dir" default="$(find twizy_sensor_kit_description)/config"/>
     <!--
@@ -11,5 +11,5 @@
     <xacro:property name="calibration" value="${xacro.load_yaml('/home/robin/Documents/autoware/install/twizy_sensor_kit_description/share/twizy_sensor_kit_description/config/sensor_kit_calibration.yaml')}"/>
     <!-- chassis from sd_twizy_base -->
-    <xacro:sd_twizy_base name="twizy_vehicle"/>
+    <!--=<xacro:sd_twizy_base name="twizy_vehicle"/>-->
       <!-- Camera -->
     <xacro:blackfly_camera frlr_prefix="front" lrc_prefix="left" parent="chassis"

File: twizy_sensor_kit_description/urdf/sensors.xacro (robot description, xacro)
@@ -10,5 +10,5 @@
   <xacro:include filename="sensor_kit.xacro"/>
   <xacro:include filename="$(find twizy_vehicle_description)/urdf/bases/sd_twizy_body.urdf.xacro"/>
-  <xacro:sd_twizy_base name="twizy_vehicle"/>
+ <!-- <xacro:sd_twizy_base name="twizy_vehicle"/>-->
   <!-- <xacro:chassis
     parent="chassis_joint"
